File: schematic/Clock.sch (KiCad schematic (older format))
At the start: 31 parts

Commit message: Clock generation mostly complete. Some inter-module connections fixed.
Parts:
- removed C? (x2): 100nF, Capacitor_SMD:C_0603_1608Metric, symbol Device:C
- removed L? (x2): 10 Ohm@100MHz, Inductor_SMD:L_0805_2012Metric, symbol Device:L_Core_Ferrite
- added C? (x4): 10nF, Capacitor_SMD:C_0603_1608Metric, symbol Device:C
- added C? (x8): 10uF, Capacitor_SMD:C_0603_1608Metric, symbol Device:C
- added C?: 220uF/10V, Capacitor_SMD:C_Elec_8x6.2, symbol Device:CP
- added C?: 1uF, Capacitor_SMD:C_0603_1608Metric, symbol Device:C
- added L?: 10 Ohm@100MHz, Inductor_SMD:L_0805_2012Metric, symbol Device:L_Core_Ferrite
- added R?: 22, Resistor_SMD:R_0603_1608Metric, symbol Device:R
- added U? (x2): TPS79333-EP, Package_TO_SOT_SMD:SOT-23-5, symbol Regulator_Linear:TPS79333-EP
- U?: value TPS79318-EP -> TPS73618DBVR
Connections:
- net labels added: +1V8_VDDCLK, +3V3_CLKOUT, +3V3_VDDACLK, +3V3_VDDOSC, +5V, CLKOUT3, MISO, MOSI, SCLK, ~CS~, ~RST~
- net labels removed: +3V3CLK, +3V3_CLK, +3V3_VDD
- wire segments 90 -> 161
Other:
- moved on the sheet: C?, L?, R?, U?, Y?
