File: schematic/Control.sch (KiCad schematic (older format))
At the start: 0 parts

Commit message: Clock generation mostly complete. Some inter-module connections fixed.
Changed lines of the file:
@@
 $Descr A4 11693 8268
 encoding utf-8
-Sheet 6 7
+Sheet 4 6
 Title ""
 Date ""
@@
 SCLK
 Text HLabel 6550 3900 0    50   Output ~ 0
-~CS_DAC_L~
+~CS_DACL~
 Text HLabel 6550 4000 0    50   Output ~ 0
-~CS_DAC_R~
+~CS_DACR~
 Text HLabel 6550 4100 0    50   Output ~ 0
 ~CS_FPGA~
+Text HLabel 6550 4200 0    50   Output ~ 0
+~CS_CLK~
 $EndSCHEMATC
