File: schematic/Control/Clock.sch (KiCad schematic (older format))
At the start: 45 parts

Commit message: Control board diagram complete at high level - Clock, USB, Control, Power and IO done. Remaining is FPGA pin assignment which will be done later to optimize board layout.
Parts:
- removed L?: 10 Ohm@100MHz, Inductor_SMD:L_0805_2012Metric, symbol Device:L_Core_Ferrite
- removed U?: TPS73618DBVR, Package_TO_SOT_SMD:SOT-23-5, symbol Regulator_Linear:TPS79318-EP
- removed U?: TPS79333-EP, Package_TO_SOT_SMD:SOT-23-5, symbol Regulator_Linear:TPS79333-EP
- added J? (x2): SMA F ST PCB, Connector_Coaxial:SMA_Amphenol_132134_Vertical, symbol Connector:Conn_Coaxial
- added U?: TPS73618DCQ, Package_TO_SOT_SMD:SOT-223-6_TabPin3, symbol Zmei_elements:TPS73601DCQ
- added U?: TPS73633DCQ, Package_TO_SOT_SMD:SOT-223-6_TabPin3, symbol Zmei_elements:TPS73601DCQ
Connections:
- net +1V8_VDDCLK: now also U?.2 (OUT)
- net +3V3_VDDACLK: now also U?.2 (OUT)
- net +5V: now also U?.1 (IN), U?.1 (IN), U?.5 (EN), U?.5 (EN)
- net CLKOUT1: now also J?.1 (In)
- net CLKOUT2: now also J?.1 (In)
- net GND: now also J?.2 (Ext), J?.2 (Ext), U?.3 (GND), U?.3 (GND)
- net at C?.2: now also U?.4 (FB) (x2)

Commit message: Provision for SPI Slave FPGA bitstream download. Switch RAM from x16 to x8 one.
Parts:
- gave numbers to parts that had none: 46
Connections:
- net +1V8_VDDCLK: now also C212.2, U203.26 (VDDS)
- net at U203.18 (VDDO0): now also C210.1, L203.1
- net at U203.20 (OUT0): now also R201.1
- net at U203.36 (OUT3): no longer R201.1
- net at U203.4 (X1), Y201.2: now also U203.7 (X2), Y201.4
- net CLKOUT3 renamed CLKOUT0
- now unconnected: U203.34 (VDDO3)
Other:
- moved on the sheet: C201, C202, C203, C204, C205, C206, C207, C208, C209, C210, C211, C212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
