File: schematic/DAC/PCM1794/PCM1794.kicad_pcb (KiCad board)
At the start: 2 copper layers, 65 x 50 mm, 62 parts, among them J101 In, J102 Out, J103 SMA F ST PCB, Q101 2SK208, Q102 BCX53-16, Q103 BCX53-16, Q104 BCX53-16, U101 PCM1792A, U102 TPS73633DCQ, U103 TL431PK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

Commit message: Send for manufacturing Control and DAC1794 boards.
Other:
- board text added: "DeWille-PCM1794 Rev. 1.0"
Changed lines of the file:
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@@
   (general
     (thickness 1.6)
-    (drawings 33)
+    (drawings 34)
     (tracks 479)
     (zones 0)
@@
   (page A4)
   (layers
-    (0 F.Cu signal)
+    (0 F.Cu signal hide)
     (31 B.Cu signal hide)
     (32 B.Adhes user hide)
@@
     (37 F.SilkS user)
     (38 B.Mask user hide)
-    (39 F.Mask user hide)
+    (39 F.Mask user)
     (40 Dwgs.User user hide)
     (41 Cmts.User user)
@@
   )
   (setup
-    (last_trace_width 0.381)
+    (last_trace_width 0.25)
     (user_trace_width 0.2032)
     (user_trace_width 0.254)
@@
     (visible_elements FEFDFF7F)
     (pcbplotparams
-      (layerselection 0x010fc_ffffffff)
-      (usegerberextensions false)
+      (layerselection 0x010f0_ffffffff)
+      (usegerberextensions true)
       (usegerberattributes false)
       (usegerberadvancedattributes false)
@@
       (outputformat 1)
       (mirror false)
-      (drillshape 1)
+      (drillshape 0)
       (scaleselection 1)
-      (outputdirectory ""))
+      (outputdirectory "../../../Fabrication/DAC_PCM1794/Gerber/"))
   )
   (net 0 "")
@@
     )
   )
+  (gr_text "DeWille-PCM1794\nRev. 1.0" (at 32.385 12.446) (layer F.SilkS)
+    (effects (font (size 1.27 1.27) (thickness 0.254)) (justify right))
+  )
   (gr_text In (at -27.813 -14.351) (layer F.SilkS)
     (effects (font (size 1.27 1.27) (thickness 0.254)))
@@
     (effects (font (size 1.016 1.016) (thickness 0.2032)))
   )
-  (gr_text -15V (at 27.686 10.922) (layer F.SilkS)
+  (gr_text -15V (at 23.114 8.89) (layer F.SilkS)
     (effects (font (size 1.016 1.016) (thickness 0.2032)))
   )
@@
     (effects (font (size 1.016 1.016) (thickness 0.2032)))
   )
-  (gr_text +15V (at 27.559 -11.303) (layer F.SilkS)
+  (gr_text +15V (at 22.987 -8.89) (layer F.SilkS)
     (effects (font (size 1.016 1.016) (thickness 0.2032)))
   )
