File: schematic/Base/DeWille_Base.kicad_pcb (KiCad board)
At the start: 2 copper layers, 200 x 200 mm, 82 parts, among them J101 HN2x10, J102 HN2x10, J103 HN2x10, J201 Conn_01x03, Q201 TIP42C, Q202 TIP42C, Q203 TIP41C, Q204 BCP56, Q205 BCP56, Q206 BCP53, U201 TL431PK, U202 TL431PK, U203 TL431PK

Commit message: Base schematic complete
Parts:
- removed J103: HN2x10, Connector_PinHeader_2.54mm:PinHeader_2x10_P2.54mm_Vertical
- removed L101: 100 Ohm@100MHz, Inductor_SMD:L_0805_2012Metric
- added B101: DeWille_Control, Zmei_Footprints:DeWille_Control, F.Cu at (-75.0, 65.0)
- added B102: DeWille_DAC, Zmei_Footprints:DeWille_DAC, F.Cu at (7.50, 42.5)
- added B103: DeWille_DAC, Zmei_Footprints:DeWille_DAC, F.Cu at (7.50, 95.0)
- added B104: DeWille_ItoV, Zmei_Footprints:DeWille_ItoV, F.Cu at (75.0, 42.5)
- added B105: DeWille_ItoV, Zmei_Footprints:DeWille_ItoV, F.Cu at (75.0, 95.0)
- added C228: 2.2uF, Capacitor_SMD:C_0603_1608Metric, F.Cu at (-106.1, 211.9)
- added C229: 100nF, Capacitor_SMD:C_0603_1608Metric, F.Cu at (-81.6, 198.0)
- added C230: 100uF/10V, Capacitor_SMD:C_Elec_6.3x5.4, F.Cu at (-103.2, 206.5)
- added C231: 10uF, Capacitor_SMD:C_0603_1608Metric, F.Cu at (-86.2, 202.6)
- added C232: 10nF, Capacitor_SMD:C_0603_1608Metric, F.Cu at (-81.6, 195.5)
- added C233: 100nF, Capacitor_SMD:C_0603_1608Metric, F.Cu at (-106.1, 214.4)
- added C234: 10uF, Capacitor_SMD:C_0603_1608Metric, F.Cu at (-102.1, 212.7)
- added C235: 100uF/10V, Capacitor_SMD:C_Elec_6.3x5.4, F.Cu at (-93.1, 198.3)
- added C301: 100nF, Capacitor_SMD:C_0603_1608Metric, F.Cu at (-91.0, 184.4)
- added C302: 100nF, Capacitor_SMD:C_0603_1608Metric, F.Cu at (-95.4, 187.3)
- added C303: 100nF, Capacitor_SMD:C_0603_1608Metric, F.Cu at (-86.6, 181.4)
- added C304: 100nF, Capacitor_SMD:C_0603_1608Metric, F.Cu at (-95.4, 189.8)
- added C305: 100nF, Capacitor_SMD:C_0603_1608Metric, F.Cu at (-79.2, 172.9)
- added C306: 100nF, Capacitor_SMD:C_0603_1608Metric, F.Cu at (-91.0, 186.9)
- added J301: I2S1, Connector_PinSocket_2.54mm:PinSocket_1x06_P2.54mm_Vertical, F.Cu at (-113.5, 171.1)
- added J302: I2S2, Connector_PinSocket_2.54mm:PinSocket_1x06_P2.54mm_Vertical, F.Cu at (-108.9, 171.1)
- added J303: SPDIF1, Connector_PinSocket_2.54mm:PinSocket_1x03_P2.54mm_Vertical, F.Cu at (-104.3, 182.5)
- added J304: SPDIF2, Connector_PinSocket_2.54mm:PinSocket_1x03_P2.54mm_Vertical, F.Cu at (-99.7, 182.5)
- added JP201: Jumper_NO_Small, Connector_PinSocket_2.54mm:PinSocket_1x02_P2.54mm_Vertical, F.Cu at (-85.8, 196.5)
- added L201: 18uH, Inductor_THT:L_Radial_D7.5mm_P3.50mm_Fastron_07P, F.Cu at (-95.3, 206.9)
- added L301: 100 Ohm@100MHz, Inductor_SMD:L_0805_2012Metric, F.Cu at (-113.6, 187.5)
- added L302: 100 Ohm@100MHz, Inductor_SMD:L_0805_2012Metric, F.Cu at (-109.2, 187.5)
- added L303: 100 Ohm@100MHz, Inductor_SMD:L_0805_2012Metric, F.Cu at (-95.2, 181.7)
- added L304: 100 Ohm@100MHz, Inductor_SMD:L_0805_2012Metric, F.Cu at (-90.8, 181.7)
- added L305: 100 Ohm@100MHz, Inductor_SMD:L_0805_2012Metric, F.Cu at (-95.2, 184.6)
- added L306: 100 Ohm@100MHz, Inductor_SMD:L_0805_2012Metric, F.Cu at (-79.0, 170.2)
- added TP301: TestPoint, TestPoint:TestPoint_Pad_D1.0mm, F.Cu at (-84.4, 184.8)
- added TP302: TestPoint, TestPoint:TestPoint_Pad_D1.0mm, F.Cu at (-87.5, 187.7)
- added TP303: TestPoint, TestPoint:TestPoint_Pad_D1.0mm, F.Cu at (-79.7, 178.8)
- added TP304: TestPoint, TestPoint:TestPoint_Pad_D1.0mm, F.Cu at (-91.9, 189.7)
- added TP305: TestPoint, TestPoint:TestPoint_Pad_D1.0mm, F.Cu at (-83.0, 181.7)
- added TP306: TestPoint, TestPoint:TestPoint_Pad_D1.0mm, F.Cu at (-79.7, 175.7)
- added TP307: TestPoint, TestPoint:TestPoint_Pad_D1.0mm, F.Cu at (-87.5, 184.7)
- added U204: AM2D-0503SZ, Zmei_Footprints:Converter_DCDC_AM2D, F.Cu at (-110.0, 196.7)
- added U205: TPS73633DCQ, Package_TO_SOT_SMD:SOT-223-6_TabPin3, F.Cu at (-103.1, 198.3)
- added U301: Si8640BB-B-IS1, Package_SO:SOIC-16_3.9x9.9mm_P1.27mm, F.Cu at (-85.5, 174.5)
- added U302: Si8640BB-B-IS1, Package_SO:SOIC-16_3.9x9.9mm_P1.27mm, F.Cu at (-93.9, 174.5)
- added U303: Si8640BB-B-IS1, Package_SO:SOIC-16_3.9x9.9mm_P1.27mm, F.Cu at (-102.4, 174.5)
- J101: value HN2x10 -> Out Left; footprint Connector_PinHeader_2.54mm:PinHeader_2x10_P2.54mm_Vertical -> TerminalBlock_Dinkle:TerminalBlock_Dinkle_DT-55-B01X-03_P10.00mm
- J102: value HN2x10 -> Out Right; footprint Connector_PinHeader_2.54mm:PinHeader_2x10_P2.54mm_Vertical -> TerminalBlock_Dinkle:TerminalBlock_Dinkle_DT-55-B01X-03_P10.00mm
- R206, R207, R218, R219, R221, R222: footprint Resistor_SMD:R_1206_3216Metric -> Resistor_SMD:R_0603_1608Metric
- moved Q204 389.1 mm to (-155.6, -34.9)
- moved U203 374.2 mm to (-144.8, -47.0)
- moved Q201 358.3 mm to (-146.1, 4.45)
- moved R213 341.3 mm to (-158.8, -46.4)
- moved R212 340.5 mm to (-138.4, -31.1)
- moved D213 336.0 mm to (-158.8, -13.3)
- moved R214 335.3 mm to (-149.2, -21.0)
- moved C222 313.0 mm to (-162.6, -22.9)
- moved R205 295.7 mm to (-141.6, -7.62)
- moved D208 290.5 mm to (-88.9, -3.17), turned to 270 degrees
- moved R220 287.6 mm to (-144.1, -22.9)
- moved R202 287.1 mm to (-90.8, -7.62)
- moved J102 277.6 mm to (115.0, 105.0), turned to 90 degrees
- moved C202 266.1 mm to (-70.5, -7.62)
- moved R217 264.0 mm to (-136.0, -19.7)
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Connections:
- C206 pad 2: Net-(C206-Pad2) -> GND
- C212 pad 2: Net-(C206-Pad2) -> GND
- C217 pad 2: Net-(C206-Pad2) -> GND
- C222 pad 2: Net-(C206-Pad2) -> GND
- C225 pad 2: Net-(C206-Pad2) -> GND
- D202 pad 2: Net-(C206-Pad2) -> GND
- D208 pad 2: Net-(C206-Pad2) -> GND
- J101 pad 1: /+5V -> Net-(B104-PadOut2)
- J101 pad 2: /SCK1 -> GND
- J101 pad 3: GND -> Net-(B104-PadOut1)
- J102 pad 1: GND -> Net-(B105-PadOut2)
- J102 pad 2: /DACL_SCK -> GND
- J102 pad 3: GND -> Net-(B105-PadOut1)
- R213 pad 2: Net-(C206-Pad2) -> GND
- R220 pad 1: Net-(C206-Pad2) -> GND
- U203 pad 2: Net-(C206-Pad2) -> GND
Other:
- board size 200 x 200 mm -> 250 x 225 mm

Commit message: Add Changes.txt, listing future changes to the schematic and boards Finish up Base board routing
Parts:
- removed C202, C203, C204: C, Capacitor_THT:C_Rect_L11.0mm_W5.1mm_P10.00mm_MKT
- removed D203, D204, D205, D206, D209, D210, D211, D212: 1N5400, Diode_THT:D_DO-27_P15.24mm_Horizontal
- removed D207, D208: SR580, Diode_THT:D_DO-27_P15.24mm_Horizontal
- removed R202, R203, R204: R, Resistor_THT:R_Axial_DIN0207_L6.3mm_D2.5mm_P10.16mm_Horizontal
- added D216: KBU8M, Diode_THT:Diode_Bridge_Vishay_KBU, F.Cu at (119.4, -73.7)
- added H101: MountingHole, MountingHole:MountingHole_3.2mm_M3_Pad, F.Cu at (-120.0, 90.0)
- added H102: MountingHole, MountingHole:MountingHole_3.2mm_M3_Pad, F.Cu at (-60.0, -95.0)
- added H103: MountingHole, MountingHole:MountingHole_3.2mm_M3_Pad, F.Cu at (120.0, 90.0)
- added H104: MountingHole, MountingHole:MountingHole_3.2mm_M3_Pad, F.Cu at (120.0, -7.50)
- added H105: MountingHole, MountingHole:MountingHole_3.2mm_M3_Pad, F.Cu at (-120.0, -7.50)
- added H106: MountingHole, MountingHole:MountingHole_3.2mm_M3_Pad, F.Cu at (40.0, -95.0)
- added H107: MountingHole, MountingHole:MountingHole_3.2mm_M3_Pad, F.Cu at (-120.0, -95.0)
- added H108: MountingHole, MountingHole:MountingHole_3.2mm_M3_Pad, F.Cu at (120.0, -95.0)
- added H109: MountingHole, MountingHole:MountingHole_3.2mm_M3_Pad, F.Cu at (-10.0, -5.00)
- added R301: 22, Resistor_SMD:R_0603_1608Metric, F.Cu at (-53.1, 76.8)
- added R302: 22, Resistor_SMD:R_0603_1608Metric, F.Cu at (-51.6, 76.8)
- added R303: 22, Resistor_SMD:R_0603_1608Metric, F.Cu at (-50.0, 76.8)
- added R304: 22, Resistor_SMD:R_0603_1608Metric, F.Cu at (-48.5, 76.8)
- added R305: 22, Resistor_SMD:R_0603_1608Metric, F.Cu at (-78.5, 76.8)
- added R306: 22, Resistor_SMD:R_0603_1608Metric, F.Cu at (-77.0, 76.8)
- added R307: 22, Resistor_SMD:R_0603_1608Metric, F.Cu at (-75.4, 76.8)
- added R308: 22, Resistor_SMD:R_0603_1608Metric, F.Cu at (-73.9, 76.8)
- added R309: 22, Resistor_SMD:R_0603_1608Metric, F.Cu at (-103.5, 75.6)
- added R310: 22, Resistor_SMD:R_0603_1608Metric, F.Cu at (-99.7, 75.6)
- added TP201: TestPoint, TestPoint:TestPoint_THTPad_D2.0mm_Drill1.0mm, F.Cu at (80.0, -57.5)
- added TP202: TestPoint, TestPoint:TestPoint_THTPad_D2.0mm_Drill1.0mm, F.Cu at (80.0, -50.0)
- D201, D202: value SR580 -> KBU8M; footprint Diode_THT:D_DO-27_P15.24mm_Horizontal -> Diode_THT:Diode_Bridge_Vishay_KBU
- TR202: value ANG_6VA -> TRAF_DUAL_SPLITPRIM; footprint Zmei_Footprints:TRAF_ANG6VA -> Zmei_Footprints:TRAF_ANG_DUAL_18_24VA
- moved C227 232.7 mm to (-19.7, -25.9), turned to 270 degrees
- moved C233 223.5 mm to (-40.8, 0.64)
- moved C228 220.5 mm to (-66.0, -4.93), turned to 90 degrees
- moved L201 215.4 mm to (-61.0, -5.71), turned to 270 degrees
- moved C234 213.9 mm to (-74.3, 0.64), turned to 90 degrees
- moved C230 212.1 mm to (-81.3, -4.45), turned to 90 degrees
- moved U204 210.4 mm to (-52.7, -5.71), turned to 90 degrees
- moved U205 206.3 mm to (-73.0, -5.71), turned to 90 degrees
- moved C229 204.5 mm to (-55.9, -4.93), turned to 90 degrees
- moved C231 202.2 mm to (-76.2, 0.64), turned to 90 degrees
- moved JP201 199.8 mm to (-86.5, -3.30), turned to 180 degrees
- moved C232 195.1 mm to (-71.8, 0.64), turned to 90 degrees
- moved TR202 193.4 mm to (42.5, -57.5), turned to 90 degrees
- moved D202 184.1 mm to (119.4, -33.7), turned to 90 degrees
- moved C226 148.7 mm to (0.00, -18.4), turned to 90 degrees
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Connections:
- B101 pad 48: (no net) -> /DACR_DATA
- C205 pad 2: Net-(C202-Pad2) -> Net-(C205-Pad2)
- C206 pad 1: Net-(C202-Pad2) -> Net-(C205-Pad2)
- C207 pad 2: Net-(C203-Pad2) -> Net-(C207-Pad2)
- C208 pad 1: Net-(C203-Pad2) -> Net-(C207-Pad1)
- C209 pad 1: GND -> Net-(C209-Pad1)
- C209 pad 2: Net-(C204-Pad2) -> GND
- C210 pad 1: Net-(C204-Pad2) -> Net-(C209-Pad1)
- C213 pad 1: Net-(C207-Pad1) -> Net-(C213-Pad1)
- C213 pad 2: Net-(C213-Pad2) -> Net-(C207-Pad2)
- C214 pad 1: Net-(C213-Pad2) -> Net-(C213-Pad1)
- C215 pad 1: GND -> Net-(C215-Pad1)
- C215 pad 2: Net-(C215-Pad2) -> GND
- C216 pad 1: Net-(C215-Pad2) -> Net-(C215-Pad1)
- C218 pad 1: Net-(C207-Pad1) -> Net-(C207-Pad2)
- D201 pad 2: Net-(C202-Pad2) -> Net-(C205-Pad2)
- D202 pad 1: Net-(C202-Pad2) -> GND
- D202 pad 2: GND -> Net-(C215-Pad1)
- D214 pad 1: Net-(C207-Pad1) -> Net-(C207-Pad2)
- J301 pad 1: Net-(J301-Pad1) -> Net-(C301-Pad2)
- J302 pad 1: /Input&Isolator/+3V3_ISOL -> Net-(C302-Pad2)
- J303 pad 1: /Input&Isolator/+3V3_ISOL -> Net-(C303-Pad2)
- J304 pad 1: /Input&Isolator/+3V3_ISOL -> Net-(C303-Pad2)
- Q202 pad 3: Net-(C207-Pad1) -> Net-(C207-Pad2)
- R206 pad 2: Net-(C207-Pad1) -> Net-(C207-Pad2)
- R215 pad 2: Net-(C207-Pad1) -> Net-(C207-Pad2)
- TR201 pad 1: Net-(TR201-Pad1) -> Net-(J201-Pad3)
- TR201 pad 11: Net-(TR201-Pad11) -> Net-(C211-Pad2)
- TR201 pad 6: Net-(TR201-Pad6) -> Net-(J201-Pad1)
- TR201 pad 8: Net-(TR201-Pad8) -> Net-(C205-Pad2)
- TR202 pad 1: Net-(TR202-Pad1) -> Net-(J201-Pad1)
- TR202 pad 4: (no net) -> Net-(TR202-Pad4)
- TR202 pad 5: Net-(TR202-Pad5) -> Net-(TR202-Pad4)
- TR202 pad 8: (no net) -> Net-(J201-Pad3)
- TR203 pad 3: Net-(C204-Pad2) -> Net-(C209-Pad1)
- TR203 pad 4: Net-(C215-Pad2) -> Net-(C215-Pad1)
- TR203 pad 5: Net-(C203-Pad2) -> Net-(C213-Pad1)
- TR203 pad 6: Net-(C213-Pad2) -> Net-(C207-Pad1)
- TR204 pad 1: Net-(J201-Pad1) -> Net-(J201-Pad3)
- TR204 pad 2: Net-(J201-Pad3) -> Net-(J201-Pad1)
- TR204 pad 3: Net-(TR204-Pad3) -> Net-(C211-Pad2)
- TR204 pad 4: Net-(TR204-Pad4) -> Net-(C205-Pad2)
- TR204 pad 5: Net-(C202-Pad2) -> Net-(TR204-Pad5)
- TR204 pad 6: Net-(C211-Pad2) -> Net-(TR204-Pad6)
- U301 pad 11: /Input&Isolator/I2S1_DATA -> Net-(R304-Pad1)
- U301 pad 12: /Input&Isolator/I2S1_LRCK -> Net-(R303-Pad1)
- U301 pad 13: /Input&Isolator/I2S1_BCK -> Net-(R302-Pad1)
- U301 pad 14: /Input&Isolator/I2S1_SCK -> Net-(R301-Pad1)
- U302 pad 11: /Input&Isolator/I2S2_DATA -> Net-(R308-Pad1)
- U302 pad 12: /Input&Isolator/I2S2_LRCK -> Net-(R307-Pad1)
- U302 pad 13: /Input&Isolator/I2S2_BCK -> Net-(R306-Pad1)
- U302 pad 14: /Input&Isolator/I2S2_SCK -> Net-(R305-Pad1)
- U303 pad 11: Net-(TP307-Pad1) -> Net-(R310-Pad1)
- U303 pad 12: /Input&Isolator/SPDIF2 -> Net-(TP307-Pad1)
- U303 pad 13: /Input&Isolator/SPDIF1 -> Net-(TP306-Pad1)
- U303 pad 14: Net-(TP306-Pad1) -> Net-(R309-Pad1)
- U303 pad 3: Net-(TP301-Pad1) -> Net-(J304-Pad2)
- U303 pad 4: Net-(J303-Pad2) -> Net-(TP301-Pad1)
- U303 pad 5: Net-(J304-Pad2) -> Net-(TP302-Pad1)
- U303 pad 6: Net-(TP302-Pad1) -> Net-(J303-Pad2)
Routing:
- net /Power Supply/+5V: track 0.00 -> 565.6 mm
- net /Power Supply/-15V: track 0.00 -> 440.7 mm, vias 0 -> 5
- net /Power Supply/+15V: track 0.00 -> 329.6 mm, vias 0 -> 4
- net GND: track 0.00 -> 273.8 mm, vias 0 -> 50
- net /Input&Isolator/+3V3_ISOL: track 0.00 -> 204.6 mm
- net /Input&Isolator/+3V3_IO: track 0.00 -> 192.3 mm
- net Net-(J201-Pad3): track 0.00 -> 122.6 mm
- net Net-(C205-Pad1): track 0.00 -> 112.4 mm
- net GNDD: track 0.00 -> 105.5 mm, vias 0 -> 10
- net Net-(C207-Pad2): track 0.00 -> 89.0 mm
- net Net-(C210-Pad2): track 0.00 -> 88.9 mm
- net /Input&Isolator/I2S1_SCK: track 0.00 -> 88.6 mm
- net Net-(J201-Pad1): track 0.00 -> 86.8 mm
- net /Input&Isolator/I2S1_BCK: track 0.00 -> 86.2 mm
- net /Input&Isolator/I2S1_LRCK: track 0.00 -> 84.3 mm
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- added copper zone on B.Cu, net GND
- added copper zone on B.Cu, net GNDD
Other:
- board size 250 x 225 mm -> 250 x 195 mm
- net class Default: clearance 0.2 -> 0.2286; via_dia 0.8 -> 0.9; via_drill 0.4 -> 0.5
- rule trace_clearance: 0.2 -> 0.2286
