File: schematic/Base/Isolator.sch (KiCad schematic (older format))
At the start: 26 parts, among them J301 I2S1, J302 I2S2, J303 SPDIF1, J304 SPDIF2, U301 Si8640BB-B-IS1, U302 Si8640BB-B-IS1, U303 Si8640BB-B-IS1

Commit message: Check-in of misc. sch changes to Base
Parts:
- added U304: Si8640BB-B-IS, Package_SO:SOIC-16W_7.5x10.3mm_P1.27mm, symbol Isolator:Si8640BB-B-IS
Changed lines of the file:
@@
 Wire Wire Line
 	3400 2050 4100 2050
+$Comp
+L Isolator:Si8640BB-B-IS U304
+U 1 1 5E904E33
+P 7800 2300
+F 0 "U304" H 7800 2967 50  0000 C CNN
+F 1 "Si8640BB-B-IS" H 7800 2876 50  0000 C CNN
+F 2 "Package_SO:SOIC-16W_7.5x10.3mm_P1.27mm" H 7800 1750 50  0001 C CIN
+F 3 "https://www.silabs.com/documents/public/data-sheets/si864x-datasheet.pdf" H 7800 2700 50  0001 C CNN
+	1    7800 2300
+	1    0    0    -1
+$EndComp
 $EndSCHEMATC

Commit message: Add Changes.txt, listing future changes to the schematic and boards Finish up Base board routing
Parts:
- removed U304: Si8640BB-B-IS, Package_SO:SOIC-16W_7.5x10.3mm_P1.27mm, symbol Isolator:Si8640BB-B-IS
- added R301, R302, R303, R304, R305, R306, R307, R308, R309, R310: 22, Resistor_SMD:R_0603_1608Metric, symbol Device:R
Connections:
- wire segments 97 -> 113
Other:
- moved on the sheet: J303, J304, TP301, TP302, TP306, TP307
